File: PCBs/Actual_PCB_Main/PCB_Main/PCB_Main.kicad_sch (KiCad schematic)
At the start: 150 parts, among them J1 fan connector, J10 To_Speaker_R, J2 10118193-0001LF, J4 10118193-0001LF, J6 XT60-M, J7 HUB75, J9 To_Speaker_L, M1 CSD17581Q3, M2 CSD17581Q3A, Q1 S8050, Q2 S8050, Q4 Fan_NMOS, Q5 S8050, Q6 S8050, SW1 SW_Push, SW2 SW_Push, SW3 SW_Push, SW4 SW_Push, U1 CP2102N-Axx-xQFN28, U2 AMS1117-3.3, U3 ESP32-WROOM-E, U4 PCM5102A, U5 LM5122MH/NOPB, U6 ESP32-WROVER-E, U7 LM4752TS, U9 CP2102N-Axx-xQFN28, Y1 CB3LV-3I-40M000000, Y2 CB3LV-3I-40M000000

Commit message: pcb almost done
Parts:
- added D2: RED LED, LED_SMD:LED_0805_2012Metric, symbol Device:LED
- added R26: 1k, Resistor_SMD:R_0805_2012Metric, symbol Device:R
Connections:
- net GND: now also R26.2; no longer C1.1, C34.1, C35.1, Cin1.1, D10.1 (K), D14.1 (K), J1.2 (Pin_2), J6.P (POS), R10.1, Rsense1.1, Ruvt1.1, Rvin1.1, U2.3 (VI), U5.4 (CSP)
- new net: D2.1 (K), R26.1
- new net VCC: C1.1, C34.1, C35.1, Cin1.1, D10.1 (K), D14.1 (K), D2.2 (A), J1.2 (Pin_2), J6.P (POS), R10.1, Rsense1.1, Ruvt1.1, Rvin1.1, U2.3 (VI), U5.4 (CSP)
Other:
- moved on the sheet: C35
Changed lines of the file:
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@@
   (junction (at 107.95 -66.04) (diameter 0) (color 0 0 0 0)
   )
+  (junction (at 29.21 17.78) (diameter 0) (color 0 0 0 0)
+  )
   (junction (at 166.37 -39.37) (diameter 0) (color 0 0 0 0)
   )
@@
   (junction (at -114.3 91.44) (diameter 0) (color 0 0 0 0)
   )
-  (junction (at 25.4 34.29) (diameter 0) (color 0 0 0 0)
-  )
   (junction (at 162.56 -74.93) (diameter 0) (color 0 0 0 0)
   )
@@
   (junction (at 78.74 17.78) (diameter 0) (color 0 0 0 0)
   )
+  (junction (at 29.21 31.75) (diameter 0) (color 0 0 0 0)
+  )
   (junction (at 190.5 -10.16) (diameter 0) (color 0 0 0 0)
   )
@@
   (junction (at -114.3 88.9) (diameter 0) (color 0 0 0 0)
   )
+  (junction (at 29.21 29.21) (diameter 0) (color 0 0 0 0)
+  )
   (junction (at 102.87 -10.16) (diameter 0) (color 0 0 0 0)
   )
@@
   (junction (at 163.83 171.45) (diameter 0) (color 0 0 0 0)
   )
+  (junction (at 29.21 20.32) (diameter 0) (color 0 0 0 0)
+  )
   (junction (at 41.91 17.78) (diameter 0) (color 0 0 0 0)
   )
@@
   (junction (at 356.87 87.63) (diameter 0) (color 0 0 0 0)
   )
-  (junction (at 25.4 26.67) (diameter 0) (color 0 0 0 0)
-  )
   (junction (at 121.92 -69.85) (diameter 0) (color 0 0 0 0)
   )
@@
   (junction (at 102.87 -69.85) (diameter 0) (color 0 0 0 0)
   )
-  (junction (at 29.21 21.59) (diameter 0) (color 0 0 0 0)
-  )
   (junction (at -36.83 68.58) (diameter 0) (color 0 0 0 0)
   )
@@
   (junction (at 134.62 -43.18) (diameter 0) (color 0 0 0 0)
   )
-  (junction (at 29.21 34.29) (diameter 0) (color 0 0 0 0)
-  )
   (junction (at 356.87 95.25) (diameter 0) (color 0 0 0 0)
   )
@@
     (stroke (width 0) (type default))
   )
+  (wire (pts (xy 31.75 20.32) (xy 29.21 20.32))
+    (stroke (width 0) (type default))
+  )
   (wire (pts (xy -39.37 73.66) (xy -36.83 73.66))
     (stroke (width 0) (type default))
@@
     (stroke (width 0) (type default))
   )
-  (wire (pts (xy 25.4 21.59) (xy 29.21 21.59))
-    (stroke (width 0) (type default))
-  )
   (wire (pts (xy 95.25 104.14) (xy 97.79 104.14))
     (stroke (width 0) (type default))
@@
     (stroke (width 0) (type default))
   )
-  (wire (pts (xy 25.4 26.67) (xy 25.4 34.29))
-    (stroke (width 0) (type default))
-  )
   (wire (pts (xy -114.3 88.9) (xy -114.3 91.44))
     (stroke (width 0) (type default))
   )
-  (wire (pts (xy 29.21 17.78) (xy 29.21 21.59))
-    (stroke (width 0) (type default))
-  )
   (wire (pts (xy 107.95 -67.31) (xy 107.95 -66.04))
     (stroke (width 0) (type default))
@@
     (stroke (width 0) (type default))
   )
+  (wire (pts (xy 29.21 31.75) (xy 29.21 34.29))
+    (stroke (width 0) (type default))
+  )
   (wire (pts (xy 443.23 100.33) (xy 449.58 100.33))
     (stroke (width 0) (type default))
@@
     (stroke (width 0) (type default))
   )
+  (wire (pts (xy 10.16 16.51) (xy 10.16 8.89))
+    (stroke (width 0) (type default))
+  )
   (wire (pts (xy 27.94 109.22) (xy 29.21 109.22))
     (stroke (width 0) (type default))
@@
     (stroke (width 0) (type default))
   )
+  (wire (pts (xy 31.75 20.32) (xy 31.75 21.59))
+    (stroke (width 0) (type default))
+  )
   (wire (pts (xy 248.92 -17.78) (xy 248.92 -19.05))
     (stroke (width 0) (type default))
@@
     (stroke (width 0) (type default))
   )
+  (wire (pts (xy 10.16 8.89) (xy 21.59 8.89))
+    (stroke (width 0) (type default))
+  )
   (wire (pts (xy 248.92 125.73) (xy 248.92 111.76))
     (stroke (width 0) (type default))
@@
     (stroke (width 0) (type default))
   )
+  (wire (pts (xy 29.21 20.32) (xy 29.21 17.78))
+    (stroke (width 0) (type default))
+  )
   (wire (pts (xy 210.82 16.51) (xy 210.82 20.32))
     (stroke (width 0) (type default))
@@
     (stroke (width 0) (type default))
   )
-  (wire (pts (xy 25.4 34.29) (xy 29.21 34.29))
-    (stroke (width 0) (type default))
-  )
   (wire (pts (xy -91.44 73.66) (xy -73.66 73.66))
     (stroke (width 0) (type default))
@@
     (stroke (width 0) (type default))
   )
+  (wire (pts (xy 29.21 29.21) (xy 31.75 29.21))
+    (stroke (width 0) (type default))
+  )
   (wire (pts (xy 162.56 24.13) (xy 168.91 24.13))
     (stroke (width 0) (type default))
@@
     (stroke (width 0) (type default))
   )
+  (wire (pts (xy 29.21 17.78) (xy 31.75 17.78))
+    (stroke (width 0) (type default))
+  )
   (wire (pts (xy 237.49 -71.12) (xy 237.49 -74.93))
     (stroke (width 0) (type default))
@@
     (stroke (width 0) (type default))
   )
+  (wire (pts (xy 29.21 17.78) (xy 21.59 17.78))
+    (stroke (width 0) (type default))
+  )
   (wire (pts (xy 190.5 -74.93) (xy 233.68 -74.93))
     (stroke (width 0) (type default))
   )
+  (wire (pts (xy 29.21 20.32) (xy 29.21 21.59))
+    (stroke (width 0) (type default))
+  )
   (wire (pts (xy 27.94 -16.51) (xy 27.94 -10.16))
     (stroke (width 0) (type default))
@@
     (stroke (width 0) (type default))
   )
-  (wire (pts (xy 29.21 24.13) (xy 29.21 34.29))
+  (wire (pts (xy 29.21 24.13) (xy 29.21 29.21))
     (stroke (width 0) (type default))
   )
@@
     (stroke (width 0) (type default))
   )
+  (wire (pts (xy 10.16 31.75) (xy 29.21 31.75))
+    (stroke (width 0) (type default))
+  )
   (wire (pts (xy 16.51 83.82) (xy 16.51 86.36))
     (stroke (width 0) (type default))
@@
     (stroke (width 0) (type default))
   )
+  (wire (pts (xy 21.59 17.78) (xy 21.59 16.51))
+    (stroke (width 0) (type default))
+  )
   (wire (pts (xy 266.7 104.14) (xy 261.62 104.14))
     (stroke (width 0) (type default))
@@
     (stroke (width 0) (type default))
   )
-  (wire (pts (xy 25.4 21.59) (xy 25.4 26.67))
-    (stroke (width 0) (type default))
-  )
   (wire (pts (xy 246.38 111.76) (xy 246.38 123.19))
     (stroke (width 0) (type default))
@@
     (stroke (width 0) (type default))
   )
+  (wire (pts (xy 29.21 29.21) (xy 29.21 31.75))
+    (stroke (width 0) (type default))
+  )
   (wire (pts (xy 238.76 116.84) (xy 266.7 116.84))
     (stroke (width 0) (type default))
@@
     (stroke (width 0) (type default))
   )
+  (wire (pts (xy 10.16 24.13) (xy 10.16 31.75))
+    (stroke (width 0) (type default))
+  )
   (wire (pts (xy 157.48 176.53) (xy 157.48 184.15))
     (stroke (width 0) (type default))
@@
     (fill (type none))
   )
-  (rectangle (start 12.7 8.89) (end 36.83 43.18)
+  (rectangle (start -1.27 3.81) (end 36.83 43.18)
     (stroke (width 0) (type default))
     (fill (type none))
@@
     (effects (font (size 1.27 1.27)) (justify left bottom))
   )
-  (text "POWER ONTO BOARD" (at 13.97 7.62 0)
+  (text "POWER ONTO BOARD" (at 13.97 3.81 0)
     (effects (font (size 1.27 1.27)) (justify left bottom))
   )
@@
     )
   )
-  (global_label "5V" (shape input) (at 29.21 21.59 0) (fields_autoplaced)
+  (global_label "5V" (shape input) (at 31.75 17.78 0) (fields_autoplaced)
     (effects (font (size 1.27 1.27)) (justify left))
-    (property "Intersheetrefs" "${INTERSHEET_REFS}" (at 34.4933 21.59 0)
+    (property "Intersheetrefs" "${INTERSHEET_REFS}" (at 37.0333 17.78 0)
       (effects (font (size 1.27 1.27)) (justify left) hide)
     )
@@
     )
   )
+  (symbol (lib_id "Device:LED") (at 21.59 12.7 270) (unit 1)
+    (in_bom yes) (on_board yes) (dnp no) (fields_autoplaced)
+    (property "Reference" "D2" (at 24.13 9.8425 90)
+      (effects (font (size 1.27 1.27)) (justify left))
+    )
+    (property "Value" "RED LED" (at 24.13 12.3825 90)
+      (effects (font (size 1.27 1.27)) (justify left))
+    )
+    (property "Footprint" "LED_SMD:LED_0805_2012Metric" (at 21.59 12.7 0)
+      (effects (font (size 1.27 1.27)) hide)
+    )
+    (property "Datasheet" "~" (at 21.59 12.7 0)
+      (effects (font (size 1.27 1.27)) hide)
+    )
+    (pin "2")
+    (pin "1")
+    (instances
+      (project "PCB_Main"
+        (path "/63211e58-9b83-4b05-a812-d0deae98b860"
+          (reference "D2") (unit 1)
+        )
+      )
+    )
+  )
   (symbol (lib_id "Device:R") (at 121.92 67.31 90) (unit 1)
     (in_bom yes) (on_board yes) (dnp no) (fields_autoplaced)
@@
     )
   )
-  (symbol (lib_id "Device:C_Polarized_US") (at 25.4 30.48 0) (unit 1)
+  (symbol (lib_id "Device:C_Polarized_US") (at 31.75 25.4 0) (unit 1)
     (in_bom yes) (on_board yes) (dnp no) (fields_autoplaced)
-    (property "Reference" "C35" (at 29.21 28.575 0)
+    (property "Reference" "C35" (at 35.56 23.495 0)
       (effects (font (size 1.27 1.27)) (justify left))
     )
-    (property "Value" "1000uF" (at 29.21 31.115 0)
+    (property "Value" "1000uF" (at 35.56 26.035 0)
       (effects (font (size 1.27 1.27)) (justify left))
     )
-    (property "Footprint" "Artisyn_Components:Audio_1000uF" (at 25.4 30.48 0)
+    (property "Footprint" "Artisyn_Components:Audio_1000uF" (at 31.75 25.4 0)
       (effects (font (size 1.27 1.27)) hide)
     )
-    (property "Datasheet" "~" (at 25.4 30.48 0)
+    (property "Datasheet" "~" (at 31.75 25.4 0)
       (effects (font (size 1.27 1.27)) hide)
     )
@@
         )
       )
+    )
+  )
+  (symbol (lib_id "Device:R") (at 10.16 20.32 0) (unit 1)
+    (in_bom yes) (on_board yes) (dnp no) (fields_autoplaced)
+    (property "Reference" "R26" (at 12.7 19.05 0)
+      (effects (font (size 1.27 1.27)) (justify left))
+    )
+    (property "Value" "1k" (at 12.7 21.59 0)
+      (effects (font (size 1.27 1.27)) (justify left))
+    )
+    (property "Footprint" "Resistor_SMD:R_0805_2012Metric" (at 8.382 20.32 90)
+      (effects (font (size 1.27 1.27)) hide)
+    )
+    (property "Datasheet" "~" (at 10.16 20.32 0)
+      (effects (font (size 1.27 1.27)) hide)
+    )
+    (pin "1")
+    (pin "2")
+    (instances
+      (project "PCB_Main"
+        (path "/63211e58-9b83-4b05-a812-d0deae98b860"
+          (reference "R26") (unit 1)
+        )
+      )

Commit message: updates to PCB
Parts:
- removed D2: RED LED, LED_SMD:LED_0805_2012Metric, symbol Device:LED
- added D3: RED LED, LED_SMD:LED_0805_2012Metric, symbol Device:LED
- added R27: 1k, Resistor_SMD:R_0805_2012Metric, symbol Device:R
- R26: value 1k -> 0
Connections:
- net 3.3V: now also D3.2 (A)
- net AGND: now also R26.2
- net GND: now also R26.1, R27.2; no longer R26.2
- net 14V: now reaches C3b1.1, Cout1.1, Coutx1.1, Csc1.1, M2.5 (DRAIN), M2.6 (DRAIN), M2.7 (DRAIN), M2.8 (DRAIN), M2.9 (DRAIN), Rfbt1.1, U7.3 (Vcc)
- new net: D3.1 (K), R27.1
Other:
- moved on the sheet: C2, C30

Commit message: PCB no errors, added PCB sandbox
Parts:
- added H5: MountingHole, MountingHole:MountingHole_2.7mm, symbol Mechanical:MountingHole
- added R28: 0, Resistor_SMD:R_0805_2012Metric, symbol Device:R
Connections:
- net AGND: now also C3b1.2, Cb1.2, Csc1.2, CsnL1.2, CsnR1.2, J10.2 (Pin_2), J9.2 (Pin_2), U7.4 (GND), R28.2
- net GND: now also R28.1; no longer C3b1.2, Cb1.2, Csc1.2, CsnL1.2, CsnR1.2, J10.2 (Pin_2), J9.2 (Pin_2), U7.4 (GND)
- net VBUS_ROVER: now also D14.1 (K); no longer D14.2 (A), D6.1 (K), R32.2
- net VBUS_WROOM: now also D10.1 (K); no longer D10.2 (A), D11.1 (K), R14.2
- net VCC: no longer D10.1 (K), D14.1 (K)
- new net: D14.2 (A), D6.1 (K), R32.2
- new net: D10.2 (A), D11.1 (K), R14.2
Other:
- moved on the sheet: R26
