File: PCBs/PCB_Main_Sandbox/PCB_Main_Sandbox.kicad_sch (KiCad schematic)
At the start: 118 parts, among them J2 XT60-M, J3 HUB75, J4 fan connector, J5 To_Speaker_L, J6 To_Speaker_R, M1 CSD17581Q3, M2 CSD17581Q3A, Q3 Fan_NMOS, SW1 SW_Push, SW2 SW_Push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

Commit message: Finished PCB sandbox design and added gbr and drl files
Parts:
- Boot2ROVER1, Boot2WROOM1: footprint Artisyn_Components:USB_TO_TTL_FT232RL -> Connector_PinSocket_2.54mm:PinSocket_1x06_P2.54mm_Vertical
Connections:
- net at Cbst1.2, L1.2, M1.5 (D1)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: now also M1.9 (Back)
Changed lines of the file:
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@@
   (junction (at 72.39 -38.1) (diameter 0) (color 0 0 0 0)
   )
+  (junction (at 163.83 -124.46) (diameter 0) (color 0 0 0 0)
+  )
   (junction (at 217.17 -130.81) (diameter 0) (color 0 0 0 0)
   )
@@
     (stroke (width 0) (type default))
   )
+  (wire (pts (xy 161.29 -124.46) (xy 163.83 -124.46))
+    (stroke (width 0) (type default))
+  )
   (wire (pts (xy 142.24 91.44) (xy 143.51 91.44))
     (stroke (width 0) (type default))
@@
     (stroke (width 0) (type default))
   )
+  (wire (pts (xy 163.83 -124.46) (xy 163.83 -123.19))
+    (stroke (width 0) (type default))
+  )
   (wire (pts (xy 185.42 13.97) (xy 175.26 13.97))
     (stroke (width 0) (type default))
@@
     (stroke (width 0) (type default))
   )
-  (wire (pts (xy 163.83 -130.81) (xy 163.83 -123.19))
+  (wire (pts (xy 163.83 -130.81) (xy 163.83 -124.46))
     (stroke (width 0) (type default))
   )
@@
     (pin "2")
     (pin "6")
+    (pin "9")
     (instances
       (project "PCB_Main_Sandbox"
@@
       (effects (font (size 1.27 1.27)))
     )
-    (property "Footprint" "Artisyn_Components:USB_TO_TTL_FT232RL" (at 444.5 -76.2 0)
+    (property "Footprint" "Connector_PinSocket_2.54mm:PinSocket_1x06_P2.54mm_Vertical" (at 444.5 -76.2 0)
       (effects (font (size 1.27 1.27)) hide)
     )
@@
       (effects (font (size 1.27 1.27)))
     )
-    (property "Footprint" "Artisyn_Components:USB_TO_TTL_FT232RL" (at 388.62 -80.01 0)
+    (property "Footprint" "Connector_PinSocket_2.54mm:PinSocket_1x06_P2.54mm_Vertical" (at 388.62 -80.01 0)
       (effects (font (size 1.27 1.27)) hide)
     )
