File: PCBs/PCB_Main_Final/PCB_Main_Final.kicad_pcb (KiCad board)
At the start: 2 copper layers, 190.5 x 63.5 mm, 119 parts, among them J10 fan connector, J13 To_Speaker_L, J14 To_Speaker_R, J7 XT60-M, J8 HUB75, J9 fan connector, M3 CSD17581Q3, M4 CSD17581Q3A, Q2 Fan_NMOS, SW8 SW_Push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

Commit message: New audio amplifier PCB
Parts:
- removed C0L3, C0R3, C3b3: 1000uF, Artisyn_Components:Audio_1000uF
- removed CiL3, CiR3, Csc3, CsnL3, CsnR7: .1uF, Capacitor_SMD:C_0805_2012Metric
- removed J13: To_Speaker_L, Connector_PinHeader_2.54mm:PinHeader_1x02_P2.54mm_Vertical
- removed J14: To_Speaker_R, Connector_PinHeader_2.54mm:PinHeader_1x02_P2.54mm_Vertical
- removed RsnL3, RsnR3: 2.7, Resistor_SMD:R_0805_2012Metric
- removed U13: LM4752TS, Artisyn_Components:LM4752
- added C0L1: 1000uF, Artisyn_Components:Audio_1000uF, F.Cu at (105.8, 114.0)
- added C0R1: 1000uF, Artisyn_Components:Audio_1000uF, F.Cu at (147.7, 100.3)
- added C3b1: 1000uF, Artisyn_Components:Audio_1000uF, F.Cu at (118.5, 103.9)
- added CiL1: .1uF, Capacitor_SMD:C_0805_2012Metric, F.Cu at (110.4, 87.4)
- added CiR1: .1uF, Capacitor_SMD:C_0805_2012Metric, F.Cu at (137.7, 88.4)
- added Csc1: .1uF, Capacitor_SMD:C_0805_2012Metric, F.Cu at (126.9, 99.1)
- added CsnL1: .1uF, Capacitor_SMD:C_0805_2012Metric, F.Cu at (127.4, 104.9)
- added CsnR2: .1uF, Capacitor_SMD:C_0805_2012Metric, F.Cu at (131.2, 99.3)
- added J5: To_Speaker_L, Connector_PinHeader_2.54mm:PinHeader_1x02_P2.54mm_Vertical, F.Cu at (96.6, 121.4)
- added J6: To_Speaker_R, Connector_PinHeader_2.54mm:PinHeader_1x02_P2.54mm_Vertical, F.Cu at (155.2, 107.2)
- added RsnL1: 2.7, Resistor_SMD:R_0805_2012Metric, F.Cu at (121.8, 97.3)
- added RsnR1: 2.7, Resistor_SMD:R_0805_2012Metric, F.Cu at (135.0, 97.3)
- added U6: LM4752TS, Artisyn_Components:LM4752, F.Cu at (126.1, 87.7)
- moved H10 29.2 mm to (148.8, 84.8)
- moved Cb3 20.7 mm to (135.9, 105.9)
- moved R33 0.15 mm to (95.8, 106.3)
Routing:
- net AGND: track 42.1 -> 204.4 mm
- net 14V: track 46.3 -> 96.2 mm, vias 0 -> 2
- net Right_Audio: track 25.4 -> 38.8 mm, vias 2 -> 3
- net Net-(J14-Pin_1): track 16.8 -> 8.78 mm
- net Net-(U13-Out_A): track 26.4 -> 20.1 mm, vias 2 -> 0
- net Net-(U13-In_A): track 24.8 -> 19.6 mm, vias 1 -> 2
- net Net-(CsnL3-Pad1): track 4.81 -> 9.97 mm, vias 0 -> 2
- net Net-(J13-Pin_1): track 6.13 -> 9.97 mm
- net Net-(U13-Bias): track 19.2 -> 15.9 mm
- net Net-(U13-In_B): track 16.2 -> 18.4 mm, vias 0 -> 2
- net Left_Audio: track 14.9 -> 13.3 mm
- net Net-(U13-Out_B): track 29.8 -> 30.4 mm
Other:
- board size 190.5 x 63.5 mm -> 190.5 x 91.9 mm

Commit message: fixed board outline and generated new GBR and DRL files
Other:
- board size 190.5 x 91.9 mm -> 190.5 x 83.8 mm
- board text added: "R1"
Changed lines of the file:
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@@
         (effects (font (size 1 1) (thickness 0.15)))
     )
-    (fp_text user "${REFERENCE}" (at -3.429 1.275 90) (layer "F.Fab")
+    (fp_text user "${REFERENCE}" (at 2.413 0.513) (layer "F.Fab")
         (effects (font (size 1 1) (thickness 0.15)))
     )
@@
     (property "SnapEDA_Link" "https://www.snapeda.com/parts/XT60-M/AMASS/view-part/?ref=snap")
     (attr through_hole)
-    (fp_text reference "J7" (at -4.825 -5.935) (layer "F.SilkS")
+    (fp_text reference "J7" (at 0.71 -2.845) (layer "F.SilkS")
         (effects (font (size 1 1) (thickness 0.15)))
     )
@@
         (effects (font (size 1 1) (thickness 0.15)))
     )
-    (fp_text user "${REFERENCE}" (at -9.144 -0.2667 90 unlocked) (layer "F.Fab")
+    (fp_text user "${REFERENCE}" (at -9.144 -0.2667 unlocked) (layer "F.Fab")
         (effects (font (size 1 1) (thickness 0.15)))
     )
@@
         (effects (font (size 1 1) (thickness 0.15)))
     )
-    (fp_text user "${REFERENCE}" (at 0.1397 -5.588 180 unlocked) (layer "F.Fab")
+    (fp_text user "${REFERENCE}" (at 0.1397 -5.588 unlocked) (layer "F.Fab")
         (effects (font (size 1 1) (thickness 0.15)))
     )
@@
         (effects (font (size 1 1) (thickness 0.15)))
     )
-    (fp_text user "WBootG" (at -3.505 5.08 180) (layer "F.Fab")
+    (fp_text user "WBootG" (at -2.235 8.865 180) (layer "F.Fab")
         (effects (font (size 1 1) (thickness 0.15)))
     )
@@
         (effects (font (size 1 1) (thickness 0.15)) (justify mirror))
     )
-    (fp_text user "${REFERENCE}" (at 2.6435 0.762 -180) (layer "B.Fab")
+    (fp_text user "${REFERENCE}" (at 1.6275 0 -180) (layer "B.Fab")
         (effects (font (size 0.5 0.5) (thickness 0.08)) (justify mirror))
     )
@@
     (property "ki_keywords" "cap capacitor")
     (attr smd)
-    (fp_text reference "Cvin2" (at 3.0275 3.302) (layer "B.SilkS")
+    (fp_text reference "Cvin2" (at 3.0275 2.54) (layer "B.SilkS")
         (effects (font (size 1 1) (thickness 0.15)) (justify mirror))
     )
@@
     )
   )
-  (gr_rect (start 43.18 42.672) (end 233.68 134.62)
-    (stroke (width 0.1) (type default)) (fill none) (layer "Edge.Cuts"))
+  (gr_line (start 233.68 48.26) (end 43.18 48.26)
+    (stroke (width 0.1) (type default)) (layer "Edge.Cuts"))
+  (gr_line (start 157.48 111.76) (end 233.68 111.76)
+    (stroke (width 0.1) (type default)) (layer "Edge.Cuts"))
+  (gr_line (start 93.98 132.08) (end 157.48 132.08)
+    (stroke (width 0.1) (type default)) (layer "Edge.Cuts"))
+  (gr_line (start 157.48 132.08) (end 157.48 111.76)
+    (stroke (width 0.1) (type default)) (layer "Edge.Cuts"))
+  (gr_line (start 93.98 111.76) (end 93.98 132.08)
+    (stroke (width 0.1) (type default)) (layer "Edge.Cuts"))
+  (gr_line (start 233.68 111.76) (end 233.68 48.26)
+    (stroke (width 0.1) (type default)) (layer "Edge.Cuts"))
+  (gr_line (start 43.18 48.26) (end 43.18 111.76)
+    (stroke (width 0.1) (type default)) (layer "Edge.Cuts"))
+  (gr_line (start 43.18 111.76) (end 93.98 111.76)
+    (stroke (width 0.1) (type default)) (layer "Edge.Cuts"))
   (gr_text "W32" (at 43.18 66.04) (layer "F.SilkS")
     (effects (font (size 1 1) (thickness 0.15)) (justify left bottom))
   )
+  (gr_text "R1" (at 43.18 68.58) (layer "F.SilkS")
+    (effects (font (size 1 1) (thickness 0.15)) (justify left bottom))
+  )
   (gr_text "21" (at 68.58 83.82) (layer "F.SilkS")
     (effects (font (size 1 1) (thickness 0.15)) (justify left bottom))
@@
   (segment (start 66.04 88.9) (end 70.395 84.545) (width 0.25) (layer "B.Cu") (net 106))
   (via (at 181.379998 68.320001) (size 3.5) (drill 3) (layers "F.Cu" "B.Cu") (net 109))
-  (via (at 126.111 82.646) (size 4.5) (drill 4) (layers "F.Cu" "B.Cu") (net 110))
+  (via (at 126.111 83.566) (size 6.5) (drill 6) (layers "F.Cu" "B.Cu") (net 110))
   (zone (net 15) (net_name "14V") (layer "F.Cu") (hatch edge 0.5)
     (priority 3)

Commit message: fixed vias and expanded boost converter
Parts:
- moved H10 38.7 mm to (160.0, 121.9)
- moved Coutx2 29.0 mm to (177.8, 127.0)
- moved Cout5 24.4 mm to (180.3, 119.4), turned to 0 degrees
Routing:
- net GND: track 226.6 -> 214.6 mm, vias 99 -> 258
- net 14V: track 96.2 -> 94.8 mm
Other:
- outline, holes or cut-outs redrawn
